File: _autosave-esp8266_pzem16_ac.kicad_pcb (KiCad board)
At the start: 2 copper layers, 26 x 24 mm, 15 parts, among them J1 RS485, J2 PWR, J3 LED, U1 ESP-12F, U2 AMS1117-3.3

Commit message: v2
Parts:
- added J4: LED, LED_SMD:LED_0805_2012Metric_Pad1.15x1.40mm_HandSolder, F.Cu at (62.2, 33.0)
- added R7: 330, Resistor_SMD:R_0805_2012Metric, F.Cu at (66.1, 33.0)
- J3: footprint -local:2pin_pad -> LED_SMD:LED_0805_2012Metric_Pad1.15x1.40mm_HandSolder
- R6: value 0 -> 330
- moved J3 1.06 mm to (66.2, 53.6), turned to 0 degrees
Connections:
- CU1 pad 5: GND -> unconnected-(CU1-Pad5)
- U1 pad 20: unconnected-(U1-Pad20) -> /GPIO_5
Routing:
- net GND: track 44.8 -> 60.5 mm
- net /GPIO_5: track 0.00 -> 7.13 mm, vias 0 -> 2
- net Net-(CU1-Pad3): track 11.2 -> 13.2 mm
- net Net-(J4-Pad1): track 0.00 -> 1.98 mm
- net +3.3V: track 41.9 -> 41.2 mm
